Commit message: updated plugin
URDF modified according to the updated plugin

File: simplecube/simplecube_description/urdf/simplecube.urdf (robot description, URDF)
Before this commit: robot simpleCube, 3 links, 2 joints
Links:
- link cube_base: geometry collision mesh filename=package://simplecube_description/meshes/qb_meshes/stl/qb_ba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; collision mesh filename=package://simplecube_description/meshes/qb_meshes/stl/qbmov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

File: softlegs/softlegs_description/urdf/leg.xacro (robot description, xacro)
@@ -159,4 +159,5 @@
         <plugin name="advanced_vsa" filename="libadvanced_plugin.so">
             <joint>${type}_ankle_shaft_joint</joint>
+            <control_type>1</control_type>
             <pub_eltau>false</pub_eltau>
             <pub_state>true</pub_state>
@@ -167,4 +168,5 @@
         <plugin name="advanced_vsa" filename="libadvanced_plugin.so">
             <joint>${type}_roll_ankle_shaft_joint</joint>
+            <control_type>1</control_type>
             <pub_eltau>false</pub_eltau>
             <pub_state>true</pub_state>

File: softlegs/softlegs_description/urdf/qb_SoftLegs.urdf.xacro (robot description, xacro)
@@ -18,5 +18,5 @@
             <origin xyz="0 0 -0.017" rpy="0 0 0"/>
             <geometry>
-				<box size="0.066 0.25 0.01" />
+				        <box size="0.066 0.25 0.01" />
             </geometry>
        </visual>
